File: hardware/neocart/adapter/prog_adapter.kicad_pcb (KiCad board)
At the start: 2 copper layers, 174 x 134 mm, 79 parts, among them J1 FPGA_U2, J2 TO_CHA, J3 FPGA_U1, J4 microSD, U1 74LVC245, U10 74HC165, U2 74LVC245, U3 74LVC245, U4 74HC165, U5 74HC165, U6 74HC165, U7 74HC165, U8 74HC165, U9 74HC165

Commit message: NeoCart final routed PCBs + JLCPCB Gerbers — ready to order
Fixed J1 GND pins (60,62,64) from QMTech schematic — FPGA now has
ground through both headers. Re-routed with Freerouting 2.0.1 (Java 21,
multi-thread). GND routed as signal net, not just copper pour.

DRC clean:
- PROG: 143 violations (121 gold finger edge + 22 text cosmetic), 0 unconnected
- CHA:  152 violations (120 gold finger edge + 32 cosmetic), 0 unconnected
- 0 starved thermals, 0 shorts, 0 clearance errors

Chip verification: all 10 ICs power correct, all signal pins connected,
J1 GND confirmed on pins 60/62/64, J2 aligned between boards.

Gerbers: neocart_prog_gerbers.zip, neocart_cha_gerbers.zip
Order settings: 2-layer, 1.6mm, ENIG, gold fingers Yes, 45° chamfer.

Co-Authored-By: Claude Opus 4.6 (1M context) <noreply@anthropic.com>
Connections:
- J1 pad 60: VCC_5V -> GND
- J1 pad 62: VCC_5V -> GND
- J1 pad 64: VCC_5V -> GND
- J3 pad 60: VCC_5V -> GND
- J3 pad 62: VCC_5V -> GND
- J3 pad 64: VCC_5V -> GND
