File: hardware/neocart/adapter/cha_adapter.kicad_pcb (KiCad board)
At the start: 2 copper layers, 173.9 x 134 mm, 53 parts, among them J2 FROM_PROG, U1 74HC165, U2 74HC165, U3 74HC165, U4 74HC165, U5 74HC165

Commit message: CHA v4 with PinSocket + PROG v5 BGA attempt
CHA v4: PinSocket footprint for J2, clean DRC (0 unconnected, 0 shorts),
LCSC fields embedded, JLCPCB plugin generates correct CPL with pad-center
coordinates. Ready for JLCPCB order.

PROG v5 BGA-256: routing failed — 122 unrouted nets after 15 passes on
two different placement attempts. Freerouting can't handle BGA fanout.
Need TQFP-144 fallback or professional BGA routing tool.

Lessons: PinSocket footprint mirrors pin 2 column. For parallel board
stacking, use PinHeader pads + socket LCSC part. JLCPCB CPL needs
pad-center coordinates (not footprint origin).

Co-Authored-By: Claude Opus 4.6 (1M context) <noreply@anthropic.com>
Parts:
- J2: footprint PinHeader_2x40_P2.54mm_Vertical -> PinSocket_2x40_P2.54mm_Vertical
- moved J2 3.00 mm to (90.0, 7.00)
